File: circuit/pocketwatch.sch (EAGLE design)
At the start: 161 parts, among them M1 MOTOR, Q1 32.768 KHz, Q2 BUZZER, Q3 MOSFET, N CHANNEL, SOT23-3, U1 ATmega645PA, U2 MCP-LI-CHARGER-1, U3 TC54, X1 USB-MICRO_B

Commit message: circuit maintainance
Parts:
- C1, C2, C3, C4: device rcl:C-EUC0603 -> pocketwatch:C-EUC0603
- C5, C6: device rcl:CPOL-USSMCA -> pocketwatch:CPOL-USSMCA
- R1, R2, R3, R4, R5, R6, R7, R8, R9: device rcl:R-US_R0603 -> pocketwatch:R-US_R0603
